File: accordeur/PB_A3.kicad_sch (KiCad schematic)
At the start: 12 parts, among them U6 LM358, U7 LM358

Commit message: Changements de Emz
Ajout de quelques footprints
Parts:
- R22, R23, R25, R27, R28, R29: footprint (none) -> Resistor_SMD:R_0805_2012Metric
Changed lines of the file:
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@@
     (property "Reference" "R29" (id 0) (at 149.86 53.34 90))
     (property "Value" "10k" (id 1) (at 149.86 55.88 90))
-    (property "Footprint" "" (id 2) (at 149.86 61.468 90)
+    (property "Footprint" "Resistor_SMD:R_0805_2012Metric" (id 2) (at 149.86 61.468 90)
       (effects (font (size 1.27 1.27)) hide)
     )
@@
     (property "Reference" "R28" (id 0) (at 125.73 66.04 90))
     (property "Value" "10k" (id 1) (at 125.73 68.58 90))
-    (property "Footprint" "" (id 2) (at 125.73 74.168 90)
+    (property "Footprint" "Resistor_SMD:R_0805_2012Metric" (id 2) (at 125.73 74.168 90)
       (effects (font (size 1.27 1.27)) hide)
     )
@@
     (property "Reference" "R27" (id 0) (at 111.76 29.21 90))
     (property "Value" "1,6k" (id 1) (at 111.76 31.75 90))
-    (property "Footprint" "" (id 2) (at 111.76 37.338 90)
+    (property "Footprint" "Resistor_SMD:R_0805_2012Metric" (id 2) (at 111.76 37.338 90)
       (effects (font (size 1.27 1.27)) hide)
     )
@@
     (property "Reference" "R22" (id 0) (at 55.88 60.96 90))
     (property "Value" "51k" (id 1) (at 55.88 63.5 90))
-    (property "Footprint" "" (id 2) (at 55.88 69.088 90)
+    (property "Footprint" "Resistor_SMD:R_0805_2012Metric" (id 2) (at 55.88 69.088 90)
       (effects (font (size 1.27 1.27)) hide)
     )
@@
     (property "Reference" "R25" (id 0) (at 88.9 63.5 90))
     (property "Value" "1,6k" (id 1) (at 88.9 66.04 90))
-    (property "Footprint" "" (id 2) (at 88.9 71.628 90)
+    (property "Footprint" "Resistor_SMD:R_0805_2012Metric" (id 2) (at 88.9 71.628 90)
       (effects (font (size 1.27 1.27)) hide)
     )
@@
     (property "Reference" "R23" (id 0) (at 72.39 36.83 90))
     (property "Value" "270k" (id 1) (at 72.39 39.37 90))
-    (property "Footprint" "" (id 2) (at 72.39 44.958 90)
-      (effects (font (size 1.27 1.27)) hide)
-    )
+    (property "Footprint" "Resistor_SMD:R_0805_2012Metric" (id 2) (at 72.39 44.958 90)
+      (effects (font (size 1.27 1.27)) hide)
+    )

Commit message: Finalisation de la rev 0 du PCB
Parts:
- removed R27: 1,6k, Resistor_SMD:R_0805_2012Metric, symbol Device:R
- added RV3: 10k, POT:POT_emz_marc, symbol Device:R_Potentiometer
- C10, C11: footprint (none) -> Capacitor_THT:CP_Radial_D5.0mm_P2.50mm
- R24, R26: footprint (none) -> Resistor_SMD:R_0805_2012Metric
Connections:
- net at R29.2, U7.1: now also RV3.2
- net at C10.1, R22.2, R23.1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: now also RV3.1
- net VCC renamed +5V
- net VEE renamed -5V
- no-connect marks 0 -> 1
Changed lines of the file:
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@@
   (junction (at 82.55 69.85) (diameter 0) (color 0 0 0 0)
   )
+  (no_connect (at 118.11 35.56))
   (wire (pts (xy 105.41 57.15) (xy 97.79 57.15))
     (stroke (width 0) (type default) (color 0 0 0 0))
@@
     (stroke (width 0) (type default) (color 0 0 0 0))
   )
+  (wire (pts (xy 123.19 132.08) (xy 123.19 134.62))
+    (stroke (width 0) (type default) (color 0 0 0 0))
+  )
   (wire (pts (xy 134.62 77.47) (xy 137.16 77.47))
     (stroke (width 0) (type default) (color 0 0 0 0))
@@
     (stroke (width 0) (type default) (color 0 0 0 0))
   )
-  (wire (pts (xy 158.75 35.56) (xy 158.75 59.69))
+  (wire (pts (xy 158.75 29.21) (xy 158.75 59.69))
     (stroke (width 0) (type default) (color 0 0 0 0))
   )
@@
     (stroke (width 0) (type default) (color 0 0 0 0))
   )
+  (wire (pts (xy 118.11 35.56) (xy 115.57 35.56))
+    (stroke (width 0) (type default) (color 0 0 0 0))
+  )
   (wire (pts (xy 76.2 43.18) (xy 82.55 43.18))
     (stroke (width 0) (type default) (color 0 0 0 0))
@@
     (stroke (width 0) (type default) (color 0 0 0 0))
   )
+  (wire (pts (xy 69.85 132.08) (xy 69.85 134.62))
+    (stroke (width 0) (type default) (color 0 0 0 0))
+  )
   (wire (pts (xy 113.03 57.15) (xy 118.11 57.15))
     (stroke (width 0) (type default) (color 0 0 0 0))
@@
     (stroke (width 0) (type default) (color 0 0 0 0))
   )
-  (wire (pts (xy 115.57 35.56) (xy 158.75 35.56))
-    (stroke (width 0) (type default) (color 0 0 0 0))
-  )
   (wire (pts (xy 114.3 99.06) (xy 106.68 99.06))
     (stroke (width 0) (type default) (color 0 0 0 0))
@@
     (stroke (width 0) (type default) (color 0 0 0 0))
   )
+  (wire (pts (xy 111.76 31.75) (xy 111.76 29.21))
+    (stroke (width 0) (type default) (color 0 0 0 0))
+  )
+  (wire (pts (xy 111.76 29.21) (xy 158.75 29.21))
+    (stroke (width 0) (type default) (color 0 0 0 0))
+  )
   (wire (pts (xy 99.06 74.93) (xy 96.52 74.93))
     (stroke (width 0) (type default) (color 0 0 0 0))
@@
   (wire (pts (xy 146.05 59.69) (xy 133.35 59.69))
     (stroke (width 0) (type default) (color 0 0 0 0))
-  )
-  (global_label "VEE" (shape input) (at 69.85 132.08 270) (fields_autoplaced)
-    (effects (font (size 1.27 1.27)) (justify right))
-    (property "Intersheet References" "${INTERSHEET_REFS}" (id 0) (at 69.7706 137.8798 90)
-      (effects (font (size 1.27 1.27)) (justify right) hide)
-    )
-  )
-  (global_label "VCC" (shape input) (at 123.19 116.84 90) (fields_autoplaced)
-    (effects (font (size 1.27 1.27)) (justify left))
-    (property "Intersheet References" "${INTERSHEET_REFS}" (id 0) (at 123.1106 110.7983 90)
-      (effects (font (size 1.27 1.27)) (justify left) hide)
-    )
-  )
-  (global_label "VEE" (shape input) (at 123.19 132.08 270) (fields_autoplaced)
-    (effects (font (size 1.27 1.27)) (justify right))
-    (property "Intersheet References" "${INTERSHEET_REFS}" (id 0) (at 123.1106 137.8798 90)
-      (effects (font (size 1.27 1.27)) (justify right) hide)
-    )
-  )
-  (global_label "VCC" (shape input) (at 69.85 116.84 90) (fields_autoplaced)
-    (effects (font (size 1.27 1.27)) (justify left))
-    (property "Intersheet References" "${INTERSHEET_REFS}" (id 0) (at 69.7706 110.7983 90)
-      (effects (font (size 1.27 1.27)) (justify left) hide)
-    )
   )
   (hierarchical_label "v_PB_A3" (shape output) (at 114.3 99.06 0)
@@
     (pin "2")
   )
+  (symbol (lib_id "power:-5V") (at 123.19 134.62 180) (unit 1)
+    (in_bom yes) (on_board yes) (fields_autoplaced)
+    (property "Reference" "#PWR053" (id 0) (at 123.19 137.16 0)
+      (effects (font (size 1.27 1.27)) hide)
+    )
+    (property "Value" "-5V" (id 1) (at 125.73 135.8899 0)
+      (effects (font (size 1.27 1.27)) (justify right))
+    )
+    (property "Footprint" "" (id 2) (at 123.19 134.62 0)
+      (effects (font (size 1.27 1.27)) hide)
+    )
+    (property "Datasheet" "" (id 3) (at 123.19 134.62 0)
+      (effects (font (size 1.27 1.27)) hide)
+    )
+    (pin "1")
+  )
   (symbol (lib_id "power:GND") (at 90.17 96.52 0) (unit 1)
     (in_bom yes) (on_board yes) (fields_autoplaced)
@@
     (property "Reference" "C10" (id 0) (at 72.39 46.99 90))
     (property "Value" "1u" (id 1) (at 72.39 49.53 90))
-    (property "Footprint" "" (id 2) (at 76.2 53.6448 0)
+    (property "Footprint" "Capacitor_THT:CP_Radial_D5.0mm_P2.50mm" (id 2) (at 76.2 53.6448 0)
       (effects (font (size 1.27 1.27)) hide)
     )
@@
     (property "Reference" "C11" (id 0) (at 109.22 49.53 90))
     (property "Value" "1u" (id 1) (at 109.22 52.07 90))
-    (property "Footprint" "" (id 2) (at 113.03 56.1848 0)
+    (property "Footprint" "Capacitor_THT:CP_Radial_D5.0mm_P2.50mm" (id 2) (at 113.03 56.1848 0)
       (effects (font (size 1.27 1.27)) hide)
     )
@@
     (property "Reference" "R26" (id 0) (at 99.06 104.14 90))
     (property "Value" "R" (id 1) (at 99.06 106.68 90))
-    (property "Footprint" "" (id 2) (at 99.06 112.268 90)
+    (property "Footprint" "Resistor_SMD:R_0805_2012Metric" (id 2) (at 99.06 112.268 90)
       (effects (font (size 1.27 1.27)) hide)
     )
@@
     (pin "1")
   )
+  (symbol (lib_id "power:-5V") (at 69.85 134.62 180) (unit 1)
+    (in_bom yes) (on_board yes) (fields_autoplaced)
+    (property "Reference" "#PWR051" (id 0) (at 69.85 137.16 0)
+      (effects (font (size 1.27 1.27)) hide)
+    )
+    (property "Value" "-5V" (id 1) (at 72.39 135.8899 0)
+      (effects (font (size 1.27 1.27)) (justify right))
+    )
+    (property "Footprint" "" (id 2) (at 69.85 134.62 0)
+      (effects (font (size 1.27 1.27)) hide)
+    )
+    (property "Datasheet" "" (id 3) (at 69.85 134.62 0)
+      (effects (font (size 1.27 1.27)) hide)
+    )
+    (pin "1")
+  )
+  (symbol (lib_id "power:+5V") (at 69.85 116.84 0) (unit 1)
+    (in_bom yes) (on_board yes) (fields_autoplaced)
+    (property "Reference" "#PWR050" (id 0) (at 69.85 120.65 0)
+      (effects (font (size 1.27 1.27)) hide)
+    )
+    (property "Value" "+5V" (id 1) (at 69.85 111.76 0))
+    (property "Footprint" "" (id 2) (at 69.85 116.84 0)
+      (effects (font (size 1.27 1.27)) hide)
+    )
+    (property "Datasheet" "" (id 3) (at 69.85 116.84 0)
+      (effects (font (size 1.27 1.27)) hide)
+    )
+    (pin "1")
+  )
   (symbol (lib_id "Amplifier_Operational:LM358") (at 144.78 74.93 0) (unit 1)
     (in_bom yes) (on_board yes) (fields_autoplaced)
@@
     (pin "1")
   )
-  (symbol (lib_id "Device:R") (at 111.76 35.56 90) (unit 1)
-    (in_bom yes) (on_board yes) (fields_autoplaced)
-    (property "Reference" "R27" (id 0) (at 111.76 29.21 90))
-    (property "Value" "1,6k" (id 1) (at 111.76 31.75 90))
-    (property "Footprint" "Resistor_SMD:R_0805_2012Metric" (id 2) (at 111.76 37.338 90)
-      (effects (font (size 1.27 1.27)) hide)
-    )
-    (property "Datasheet" "~" (id 3) (at 111.76 35.56 0)
-      (effects (font (size 1.27 1.27)) hide)
-    )
-    (pin "1")
-    (pin "2")
-  )
   (symbol (lib_id "Amplifier_Operational:LM358") (at 99.06 99.06 0) (unit 2)
     (in_bom yes) (on_board yes) (fields_autoplaced)
@@
     (pin "7")
   )
+  (symbol (lib_id "power:+5V") (at 123.19 116.84 0) (unit 1)
+    (in_bom yes) (on_board yes) (fields_autoplaced)
+    (property "Reference" "#PWR052" (id 0) (at 123.19 120.65 0)
+      (effects (font (size 1.27 1.27)) hide)
+    )
+    (property "Value" "+5V" (id 1) (at 123.19 111.76 0))
+    (property "Footprint" "" (id 2) (at 123.19 116.84 0)
+      (effects (font (size 1.27 1.27)) hide)
+    )
+    (property "Datasheet" "" (id 3) (at 123.19 116.84 0)
+      (effects (font (size 1.27 1.27)) hide)
+    )
+    (pin "1")
+  )
+  (symbol (lib_id "Device:R_Potentiometer") (at 111.76 35.56 90) (unit 1)
+    (in_bom yes) (on_board yes) (fields_autoplaced)
+    (property "Reference" "RV3" (id 0) (at 111.76 39.37 90))
+    (property "Value" "10k" (id 1) (at 111.76 41.91 90))
+    (property "Footprint" "POT:POT_emz_marc" (id 2) (at 111.76 35.56 0)
+      (effects (font (size 1.27 1.27)) hide)
+    )
+    (property "Datasheet" "~" (id 3) (at 111.76 35.56 0)
+      (effects (font (size 1.27 1.27)) hide)
+    )
+    (pin "1")
+    (pin "2")
+    (pin "3")
+  )
   (symbol (lib_id "Amplifier_Operational:LM358") (at 72.39 124.46 0) (unit 3)
     (in_bom yes) (on_board yes) (fields_autoplaced)
@@
     (property "Reference" "R24" (id 0) (at 86.36 95.25 90))
     (property "Value" "R" (id 1) (at 86.36 97.79 90))
-    (property "Footprint" "" (id 2) (at 86.36 103.378 90)
-      (effects (font (size 1.27 1.27)) hide)
-    )
+    (property "Footprint" "Resistor_SMD:R_0805_2012Metric" (id 2) (at 86.36 103.378 90)
+      (effects (font (size 1.27 1.27)) hide)
+    )

Commit message: Checkpoint dernier review PCB
Parts:
- R22: value 51k -> 1,22k
- R24: value R -> 1k
- R25: value 1,6k -> 1k
- R26: value R -> 4,3k
- RV3: value 10k -> 1k
Changed lines of the file:
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@@
     (in_bom yes) (on_board yes) (fields_autoplaced)
     (property "Reference" "R26" (id 0) (at 99.06 104.14 90))
-    (property "Value" "R" (id 1) (at 99.06 106.68 90))
+    (property "Value" "4,3k" (id 1) (at 99.06 106.68 90))
     (property "Footprint" "Resistor_SMD:R_0805_2012Metric" (id 2) (at 99.06 112.268 90)
       (effects (font (size 1.27 1.27)) hide)
@@
     (in_bom yes) (on_board yes) (fields_autoplaced)
     (property "Reference" "RV3" (id 0) (at 111.76 39.37 90))
-    (property "Value" "10k" (id 1) (at 111.76 41.91 90))
+    (property "Value" "1k" (id 1) (at 111.76 41.91 90))
     (property "Footprint" "POT:POT_emz_marc" (id 2) (at 111.76 35.56 0)
       (effects (font (size 1.27 1.27)) hide)
@@
     (in_bom yes) (on_board yes) (fields_autoplaced)
     (property "Reference" "R22" (id 0) (at 55.88 60.96 90))
-    (property "Value" "51k" (id 1) (at 55.88 63.5 90))
+    (property "Value" "1,22k" (id 1) (at 55.88 63.5 90))
     (property "Footprint" "Resistor_SMD:R_0805_2012Metric" (id 2) (at 55.88 69.088 90)
       (effects (font (size 1.27 1.27)) hide)
@@
     (in_bom yes) (on_board yes) (fields_autoplaced)
     (property "Reference" "R25" (id 0) (at 88.9 63.5 90))
-    (property "Value" "1,6k" (id 1) (at 88.9 66.04 90))
+    (property "Value" "1k" (id 1) (at 88.9 66.04 90))
     (property "Footprint" "Resistor_SMD:R_0805_2012Metric" (id 2) (at 88.9 71.628 90)
       (effects (font (size 1.27 1.27)) hide)
@@
     (in_bom yes) (on_board yes) (fields_autoplaced)
     (property "Reference" "R24" (id 0) (at 86.36 95.25 90))
-    (property "Value" "R" (id 1) (at 86.36 97.79 90))
+    (property "Value" "1k" (id 1) (at 86.36 97.79 90))
     (property "Footprint" "Resistor_SMD:R_0805_2012Metric" (id 2) (at 86.36 103.378 90)
       (effects (font (size 1.27 1.27)) hide)

Commit message: Finalisation du placement des pièces
Prochaine étape : routing
Parts:
- R22, R23, R24, R25, R26, R28, R29: footprint Resistor_SMD:R_0805_2012Metric -> Resistor_SMD:R_0805_2012Metric_Pad1.20x1.40mm_HandSolder
Changed lines of the file:
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@@
     (property "Reference" "R29" (id 0) (at 149.86 53.34 90))
     (property "Value" "10k" (id 1) (at 149.86 55.88 90))
-    (property "Footprint" "Resistor_SMD:R_0805_2012Metric" (id 2) (at 149.86 61.468 90)
+    (property "Footprint" "Resistor_SMD:R_0805_2012Metric_Pad1.20x1.40mm_HandSolder" (id 2) (at 149.86 61.468 90)
       (effects (font (size 1.27 1.27)) hide)
     )
@@
     (property "Reference" "R26" (id 0) (at 99.06 104.14 90))
     (property "Value" "4,3k" (id 1) (at 99.06 106.68 90))
-    (property "Footprint" "Resistor_SMD:R_0805_2012Metric" (id 2) (at 99.06 112.268 90)
+    (property "Footprint" "Resistor_SMD:R_0805_2012Metric_Pad1.20x1.40mm_HandSolder" (id 2) (at 99.06 112.268 90)
       (effects (font (size 1.27 1.27)) hide)
     )
@@
     (property "Reference" "R28" (id 0) (at 125.73 66.04 90))
     (property "Value" "10k" (id 1) (at 125.73 68.58 90))
-    (property "Footprint" "Resistor_SMD:R_0805_2012Metric" (id 2) (at 125.73 74.168 90)
+    (property "Footprint" "Resistor_SMD:R_0805_2012Metric_Pad1.20x1.40mm_HandSolder" (id 2) (at 125.73 74.168 90)
       (effects (font (size 1.27 1.27)) hide)
     )
@@
     (property "Reference" "R22" (id 0) (at 55.88 60.96 90))
     (property "Value" "1,22k" (id 1) (at 55.88 63.5 90))
-    (property "Footprint" "Resistor_SMD:R_0805_2012Metric" (id 2) (at 55.88 69.088 90)
+    (property "Footprint" "Resistor_SMD:R_0805_2012Metric_Pad1.20x1.40mm_HandSolder" (id 2) (at 55.88 69.088 90)
       (effects (font (size 1.27 1.27)) hide)
     )
@@
     (property "Reference" "R25" (id 0) (at 88.9 63.5 90))
     (property "Value" "1k" (id 1) (at 88.9 66.04 90))
-    (property "Footprint" "Resistor_SMD:R_0805_2012Metric" (id 2) (at 88.9 71.628 90)
+    (property "Footprint" "Resistor_SMD:R_0805_2012Metric_Pad1.20x1.40mm_HandSolder" (id 2) (at 88.9 71.628 90)
       (effects (font (size 1.27 1.27)) hide)
     )
@@
     (property "Reference" "R24" (id 0) (at 86.36 95.25 90))
     (property "Value" "1k" (id 1) (at 86.36 97.79 90))
-    (property "Footprint" "Resistor_SMD:R_0805_2012Metric" (id 2) (at 86.36 103.378 90)
+    (property "Footprint" "Resistor_SMD:R_0805_2012Metric_Pad1.20x1.40mm_HandSolder" (id 2) (at 86.36 103.378 90)
       (effects (font (size 1.27 1.27)) hide)
     )
@@
     (property "Reference" "R23" (id 0) (at 72.39 36.83 90))
     (property "Value" "270k" (id 1) (at 72.39 39.37 90))
-    (property "Footprint" "Resistor_SMD:R_0805_2012Metric" (id 2) (at 72.39 44.958 90)
-      (effects (font (size 1.27 1.27)) hide)
-    )
+    (property "Footprint" "Resistor_SMD:R_0805_2012Metric_Pad1.20x1.40mm_HandSolder" (id 2) (at 72.39 44.958 90)
+      (effects (font (size 1.27 1.27)) hide)
+    )
