File: accordeur/PB_D3.kicad_sch (KiCad schematic)
At the start: 12 parts, among them U4 LM358, U5 LM358

Commit message: Changements de Emz
Ajout de quelques footprints
Parts:
- R14, R15, R17, R19, R20, R21: footprint (none) -> Resistor_SMD:R_0805_2012Metric
Changed lines of the file:
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@@
     (property "Reference" "R19" (id 0) (at 111.76 29.21 90))
     (property "Value" "1,6k" (id 1) (at 111.76 31.75 90))
-    (property "Footprint" "" (id 2) (at 111.76 37.338 90)
+    (property "Footprint" "Resistor_SMD:R_0805_2012Metric" (id 2) (at 111.76 37.338 90)
       (effects (font (size 1.27 1.27)) hide)
     )
@@
     (property "Reference" "R21" (id 0) (at 149.86 53.34 90))
     (property "Value" "10k" (id 1) (at 149.86 55.88 90))
-    (property "Footprint" "" (id 2) (at 149.86 61.468 90)
+    (property "Footprint" "Resistor_SMD:R_0805_2012Metric" (id 2) (at 149.86 61.468 90)
       (effects (font (size 1.27 1.27)) hide)
     )
@@
     (property "Reference" "R20" (id 0) (at 125.73 66.04 90))
     (property "Value" "10k" (id 1) (at 125.73 68.58 90))
-    (property "Footprint" "" (id 2) (at 125.73 74.168 90)
+    (property "Footprint" "Resistor_SMD:R_0805_2012Metric" (id 2) (at 125.73 74.168 90)
       (effects (font (size 1.27 1.27)) hide)
     )
@@
     (property "Reference" "R15" (id 0) (at 72.39 36.83 90))
     (property "Value" "270k" (id 1) (at 72.39 39.37 90))
-    (property "Footprint" "" (id 2) (at 72.39 44.958 90)
+    (property "Footprint" "Resistor_SMD:R_0805_2012Metric" (id 2) (at 72.39 44.958 90)
       (effects (font (size 1.27 1.27)) hide)
     )
@@
     (property "Reference" "R17" (id 0) (at 88.9 63.5 90))
     (property "Value" "1,6k" (id 1) (at 88.9 66.04 90))
-    (property "Footprint" "" (id 2) (at 88.9 71.628 90)
+    (property "Footprint" "Resistor_SMD:R_0805_2012Metric" (id 2) (at 88.9 71.628 90)
       (effects (font (size 1.27 1.27)) hide)
     )
@@
     (property "Reference" "R14" (id 0) (at 55.88 60.96 90))
     (property "Value" "51k" (id 1) (at 55.88 63.5 90))
-    (property "Footprint" "" (id 2) (at 55.88 69.088 90)
+    (property "Footprint" "Resistor_SMD:R_0805_2012Metric" (id 2) (at 55.88 69.088 90)
       (effects (font (size 1.27 1.27)) hide)
     )

Commit message: Finalisation de la rev 0 du PCB
Parts:
- removed R19: 1,6k, Resistor_SMD:R_0805_2012Metric, symbol Device:R
- added RV2: 10k, POT:POT_emz_marc, symbol Device:R_Potentiometer
- C8, C9: footprint (none) -> Capacitor_THT:CP_Radial_D5.0mm_P2.50mm
- R16, R18: footprint (none) -> Resistor_SMD:R_0805_2012Metric
Connections:
- net at C8.1, R14.2, R15.1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: now also RV2.1
- net at R21.2, U5.1: now also RV2.2
- net VCC renamed +5V
- net VEE renamed -5V
- no-connect marks 0 -> 1
Changed lines of the file:
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@@
   (junction (at 82.55 69.85) (diameter 0) (color 0 0 0 0)
   )
+  (no_connect (at 118.11 35.56))
   (wire (pts (xy 105.41 57.15) (xy 97.79 57.15))
     (stroke (width 0) (type default) (color 0 0 0 0))
   )
+  (wire (pts (xy 69.85 132.08) (xy 69.85 135.89))
+    (stroke (width 0) (type default) (color 0 0 0 0))
+  )
   (wire (pts (xy 63.5 54.61) (xy 63.5 67.31))
     (stroke (width 0) (type default) (color 0 0 0 0))
@@
     (stroke (width 0) (type default) (color 0 0 0 0))
   )
+  (wire (pts (xy 111.76 31.75) (xy 111.76 30.48))
+    (stroke (width 0) (type default) (color 0 0 0 0))
+  )
   (wire (pts (xy 82.55 69.85) (xy 85.09 69.85))
     (stroke (width 0) (type default) (color 0 0 0 0))
   )
+  (wire (pts (xy 118.11 35.56) (xy 115.57 35.56))
+    (stroke (width 0) (type default) (color 0 0 0 0))
+  )
   (wire (pts (xy 134.62 77.47) (xy 137.16 77.47))
     (stroke (width 0) (type default) (color 0 0 0 0))
@@
     (stroke (width 0) (type default) (color 0 0 0 0))
   )
-  (wire (pts (xy 158.75 35.56) (xy 158.75 59.69))
+  (wire (pts (xy 158.75 30.48) (xy 158.75 59.69))
     (stroke (width 0) (type default) (color 0 0 0 0))
   )
@@
     (stroke (width 0) (type default) (color 0 0 0 0))
   )
+  (wire (pts (xy 123.19 114.3) (xy 123.19 116.84))
+    (stroke (width 0) (type default) (color 0 0 0 0))
+  )
   (wire (pts (xy 97.79 69.85) (xy 99.06 69.85))
     (stroke (width 0) (type default) (color 0 0 0 0))
@@
     (stroke (width 0) (type default) (color 0 0 0 0))
   )
+  (wire (pts (xy 123.19 132.08) (xy 123.19 135.89))
+    (stroke (width 0) (type default) (color 0 0 0 0))
+  )
   (wire (pts (xy 114.3 72.39) (xy 118.11 72.39))
     (stroke (width 0) (type default) (color 0 0 0 0))
@@
     (stroke (width 0) (type default) (color 0 0 0 0))
   )
+  (wire (pts (xy 69.85 114.3) (xy 69.85 116.84))
+    (stroke (width 0) (type default) (color 0 0 0 0))
+  )
   (wire (pts (xy 81.28 69.85) (xy 82.55 69.85))
     (stroke (width 0) (type default) (color 0 0 0 0))
@@
     (stroke (width 0) (type default) (color 0 0 0 0))
   )
-  (wire (pts (xy 115.57 35.56) (xy 158.75 35.56))
-    (stroke (width 0) (type default) (color 0 0 0 0))
-  )
   (wire (pts (xy 114.3 99.06) (xy 106.68 99.06))
     (stroke (width 0) (type default) (color 0 0 0 0))
@@
     (stroke (width 0) (type default) (color 0 0 0 0))
   )
+  (wire (pts (xy 111.76 30.48) (xy 158.75 30.48))
+    (stroke (width 0) (type default) (color 0 0 0 0))
+  )
   (wire (pts (xy 133.35 72.39) (xy 137.16 72.39))
     (stroke (width 0) (type default) (color 0 0 0 0))
@@
   (wire (pts (xy 146.05 59.69) (xy 133.35 59.69))
     (stroke (width 0) (type default) (color 0 0 0 0))
-  )
-  (global_label "VEE" (shape input) (at 123.19 132.08 270) (fields_autoplaced)
-    (effects (font (size 1.27 1.27)) (justify right))
-    (property "Intersheet References" "${INTERSHEET_REFS}" (id 0) (at 123.1106 137.8798 90)
-      (effects (font (size 1.27 1.27)) (justify right) hide)
-    )
-  )
-  (global_label "VCC" (shape input) (at 123.19 116.84 90) (fields_autoplaced)
-    (effects (font (size 1.27 1.27)) (justify left))
-    (property "Intersheet References" "${INTERSHEET_REFS}" (id 0) (at 123.1106 110.7983 90)
-      (effects (font (size 1.27 1.27)) (justify left) hide)
-    )
-  )
-  (global_label "VEE" (shape input) (at 69.85 132.08 270) (fields_autoplaced)
-    (effects (font (size 1.27 1.27)) (justify right))
-    (property "Intersheet References" "${INTERSHEET_REFS}" (id 0) (at 69.7706 137.8798 90)
-      (effects (font (size 1.27 1.27)) (justify right) hide)
-    )
-  )
-  (global_label "VCC" (shape input) (at 69.85 116.84 90) (fields_autoplaced)
-    (effects (font (size 1.27 1.27)) (justify left))
-    (property "Intersheet References" "${INTERSHEET_REFS}" (id 0) (at 69.7706 110.7983 90)
-      (effects (font (size 1.27 1.27)) (justify left) hide)
-    )
   )
   (hierarchical_label "v_PB_D3" (shape output) (at 114.3 99.06 0)
@@
     (property "Reference" "R16" (id 0) (at 86.36 95.25 90))
     (property "Value" "R" (id 1) (at 86.36 97.79 90))
-    (property "Footprint" "" (id 2) (at 86.36 103.378 90)
+    (property "Footprint" "Resistor_SMD:R_0805_2012Metric" (id 2) (at 86.36 103.378 90)
       (effects (font (size 1.27 1.27)) hide)
     )
@@
     (pin "8")
   )
+  (symbol (lib_id "power:+5V") (at 69.85 114.3 0) (unit 1)
+    (in_bom yes) (on_board yes) (fields_autoplaced)
+    (property "Reference" "#PWR046" (id 0) (at 69.85 118.11 0)
+      (effects (font (size 1.27 1.27)) hide)
+    )
+    (property "Value" "+5V" (id 1) (at 69.85 109.22 0))
+    (property "Footprint" "" (id 2) (at 69.85 114.3 0)
+      (effects (font (size 1.27 1.27)) hide)
+    )
+    (property "Datasheet" "" (id 3) (at 69.85 114.3 0)
+      (effects (font (size 1.27 1.27)) hide)
+    )
+    (pin "1")
+  )
   (symbol (lib_id "Device:C") (at 109.22 57.15 90) (unit 1)
     (in_bom yes) (on_board yes) (fields_autoplaced)
     (property "Reference" "C9" (id 0) (at 109.22 49.53 90))
     (property "Value" "1u" (id 1) (at 109.22 52.07 90))
-    (property "Footprint" "" (id 2) (at 113.03 56.1848 0)
+    (property "Footprint" "Capacitor_THT:CP_Radial_D5.0mm_P2.50mm" (id 2) (at 113.03 56.1848 0)
       (effects (font (size 1.27 1.27)) hide)
     )
@@
     (property "Reference" "C8" (id 0) (at 72.39 46.99 90))
     (property "Value" "1u" (id 1) (at 72.39 49.53 90))
-    (property "Footprint" "" (id 2) (at 76.2 53.6448 0)
+    (property "Footprint" "Capacitor_THT:CP_Radial_D5.0mm_P2.50mm" (id 2) (at 76.2 53.6448 0)
       (effects (font (size 1.27 1.27)) hide)
     )
@@
     (pin "7")
   )
-  (symbol (lib_id "Device:R") (at 111.76 35.56 90) (unit 1)
-    (in_bom yes) (on_board yes) (fields_autoplaced)
-    (property "Reference" "R19" (id 0) (at 111.76 29.21 90))
-    (property "Value" "1,6k" (id 1) (at 111.76 31.75 90))
-    (property "Footprint" "Resistor_SMD:R_0805_2012Metric" (id 2) (at 111.76 37.338 90)
+  (symbol (lib_id "Device:R_Potentiometer") (at 111.76 35.56 90) (unit 1)
+    (in_bom yes) (on_board yes) (fields_autoplaced)
+    (property "Reference" "RV2" (id 0) (at 111.76 39.37 90))
+    (property "Value" "10k" (id 1) (at 111.76 41.91 90))
+    (property "Footprint" "POT:POT_emz_marc" (id 2) (at 111.76 35.56 0)
       (effects (font (size 1.27 1.27)) hide)
     )
@@
     (pin "1")
     (pin "2")
+    (pin "3")
   )
   (symbol (lib_id "Amplifier_Operational:LM358") (at 72.39 124.46 0) (unit 3)
@@
     (pin "4")
     (pin "8")
+  )
+  (symbol (lib_id "power:-5V") (at 123.19 135.89 180) (unit 1)
+    (in_bom yes) (on_board yes) (fields_autoplaced)
+    (property "Reference" "#PWR049" (id 0) (at 123.19 138.43 0)
+      (effects (font (size 1.27 1.27)) hide)
+    )
+    (property "Value" "-5V" (id 1) (at 125.73 137.1599 0)
+      (effects (font (size 1.27 1.27)) (justify right))
+    )
+    (property "Footprint" "" (id 2) (at 123.19 135.89 0)
+      (effects (font (size 1.27 1.27)) hide)
+    )
+    (property "Datasheet" "" (id 3) (at 123.19 135.89 0)
+      (effects (font (size 1.27 1.27)) hide)
+    )
+    (pin "1")
   )
   (symbol (lib_id "Device:R") (at 149.86 59.69 90) (unit 1)
@@
     (pin "1")
   )
+  (symbol (lib_id "power:-5V") (at 69.85 135.89 180) (unit 1)
+    (in_bom yes) (on_board yes) (fields_autoplaced)
+    (property "Reference" "#PWR047" (id 0) (at 69.85 138.43 0)
+      (effects (font (size 1.27 1.27)) hide)
+    )
+    (property "Value" "-5V" (id 1) (at 72.39 137.1599 0)
+      (effects (font (size 1.27 1.27)) (justify right))
+    )
+    (property "Footprint" "" (id 2) (at 69.85 135.89 0)
+      (effects (font (size 1.27 1.27)) hide)
+    )
+    (property "Datasheet" "" (id 3) (at 69.85 135.89 0)
+      (effects (font (size 1.27 1.27)) hide)
+    )
+    (pin "1")
+  )
   (symbol (lib_id "power:GND") (at 64.77 73.66 0) (unit 1)
     (in_bom yes) (on_board yes) (fields_autoplaced)
@@
     (pin "1")
   )
+  (symbol (lib_id "power:+5V") (at 123.19 114.3 0) (unit 1)
+    (in_bom yes) (on_board yes) (fields_autoplaced)
+    (property "Reference" "#PWR048" (id 0) (at 123.19 118.11 0)
+      (effects (font (size 1.27 1.27)) hide)
+    )
+    (property "Value" "+5V" (id 1) (at 123.19 109.22 0))
+    (property "Footprint" "" (id 2) (at 123.19 114.3 0)
+      (effects (font (size 1.27 1.27)) hide)
+    )
+    (property "Datasheet" "" (id 3) (at 123.19 114.3 0)
+      (effects (font (size 1.27 1.27)) hide)
+    )
+    (pin "1")
+  )
   (symbol (lib_id "Device:R") (at 99.06 110.49 90) (unit 1)
     (in_bom yes) (on_board yes) (fields_autoplaced)
     (property "Reference" "R18" (id 0) (at 99.06 104.14 90))
     (property "Value" "R" (id 1) (at 99.06 106.68 90))
-    (property "Footprint" "" (id 2) (at 99.06 112.268 90)
-      (effects (font (size 1.27 1.27)) hide)
-    )
+    (property "Footprint" "Resistor_SMD:R_0805_2012Metric" (id 2) (at 99.06 112.268 90)
+      (effects (font (size 1.27 1.27)) hide)
+    )

Commit message: Checkpoint dernier review PCB
Parts:
- R14: value 51k -> 1,22k
- R16: value R -> 1k
- R17: value 1,6k -> 1k
- R18: value R -> 4,3k
Changed lines of the file:
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@@
     (in_bom yes) (on_board yes) (fields_autoplaced)
     (property "Reference" "R16" (id 0) (at 86.36 95.25 90))
-    (property "Value" "R" (id 1) (at 86.36 97.79 90))
+    (property "Value" "1k" (id 1) (at 86.36 97.79 90))
     (property "Footprint" "Resistor_SMD:R_0805_2012Metric" (id 2) (at 86.36 103.378 90)
       (effects (font (size 1.27 1.27)) hide)
@@
     (in_bom yes) (on_board yes) (fields_autoplaced)
     (property "Reference" "R17" (id 0) (at 88.9 63.5 90))
-    (property "Value" "1,6k" (id 1) (at 88.9 66.04 90))
+    (property "Value" "1k" (id 1) (at 88.9 66.04 90))
     (property "Footprint" "Resistor_SMD:R_0805_2012Metric" (id 2) (at 88.9 71.628 90)
       (effects (font (size 1.27 1.27)) hide)
@@
     (in_bom yes) (on_board yes) (fields_autoplaced)
     (property "Reference" "R14" (id 0) (at 55.88 60.96 90))
-    (property "Value" "51k" (id 1) (at 55.88 63.5 90))
+    (property "Value" "1,22k" (id 1) (at 55.88 63.5 90))
     (property "Footprint" "Resistor_SMD:R_0805_2012Metric" (id 2) (at 55.88 69.088 90)
       (effects (font (size 1.27 1.27)) hide)
@@
     (in_bom yes) (on_board yes) (fields_autoplaced)
     (property "Reference" "R18" (id 0) (at 99.06 104.14 90))
-    (property "Value" "R" (id 1) (at 99.06 106.68 90))
+    (property "Value" "4,3k" (id 1) (at 99.06 106.68 90))
     (property "Footprint" "Resistor_SMD:R_0805_2012Metric" (id 2) (at 99.06 112.268 90)
       (effects (font (size 1.27 1.27)) hide)

Commit message: Finalisation du placement des pièces
Prochaine étape : routing
Parts:
- R14, R15, R16, R17, R18, R20, R21: footprint Resistor_SMD:R_0805_2012Metric -> Resistor_SMD:R_0805_2012Metric_Pad1.20x1.40mm_HandSolder
Changed lines of the file:
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@@
     (property "Reference" "R16" (id 0) (at 86.36 95.25 90))
     (property "Value" "1k" (id 1) (at 86.36 97.79 90))
-    (property "Footprint" "Resistor_SMD:R_0805_2012Metric" (id 2) (at 86.36 103.378 90)
+    (property "Footprint" "Resistor_SMD:R_0805_2012Metric_Pad1.20x1.40mm_HandSolder" (id 2) (at 86.36 103.378 90)
       (effects (font (size 1.27 1.27)) hide)
     )
@@
     (property "Reference" "R21" (id 0) (at 149.86 53.34 90))
     (property "Value" "10k" (id 1) (at 149.86 55.88 90))
-    (property "Footprint" "Resistor_SMD:R_0805_2012Metric" (id 2) (at 149.86 61.468 90)
+    (property "Footprint" "Resistor_SMD:R_0805_2012Metric_Pad1.20x1.40mm_HandSolder" (id 2) (at 149.86 61.468 90)
       (effects (font (size 1.27 1.27)) hide)
     )
@@
     (property "Reference" "R20" (id 0) (at 125.73 66.04 90))
     (property "Value" "10k" (id 1) (at 125.73 68.58 90))
-    (property "Footprint" "Resistor_SMD:R_0805_2012Metric" (id 2) (at 125.73 74.168 90)
+    (property "Footprint" "Resistor_SMD:R_0805_2012Metric_Pad1.20x1.40mm_HandSolder" (id 2) (at 125.73 74.168 90)
       (effects (font (size 1.27 1.27)) hide)
     )
@@
     (property "Reference" "R15" (id 0) (at 72.39 36.83 90))
     (property "Value" "270k" (id 1) (at 72.39 39.37 90))
-    (property "Footprint" "Resistor_SMD:R_0805_2012Metric" (id 2) (at 72.39 44.958 90)
+    (property "Footprint" "Resistor_SMD:R_0805_2012Metric_Pad1.20x1.40mm_HandSolder" (id 2) (at 72.39 44.958 90)
       (effects (font (size 1.27 1.27)) hide)
     )
@@
     (property "Reference" "R17" (id 0) (at 88.9 63.5 90))
     (property "Value" "1k" (id 1) (at 88.9 66.04 90))
-    (property "Footprint" "Resistor_SMD:R_0805_2012Metric" (id 2) (at 88.9 71.628 90)
+    (property "Footprint" "Resistor_SMD:R_0805_2012Metric_Pad1.20x1.40mm_HandSolder" (id 2) (at 88.9 71.628 90)
       (effects (font (size 1.27 1.27)) hide)
     )
@@
     (property "Reference" "R14" (id 0) (at 55.88 60.96 90))
     (property "Value" "1,22k" (id 1) (at 55.88 63.5 90))
-    (property "Footprint" "Resistor_SMD:R_0805_2012Metric" (id 2) (at 55.88 69.088 90)
+    (property "Footprint" "Resistor_SMD:R_0805_2012Metric_Pad1.20x1.40mm_HandSolder" (id 2) (at 55.88 69.088 90)
       (effects (font (size 1.27 1.27)) hide)
     )
@@
     (property "Reference" "R18" (id 0) (at 99.06 104.14 90))
     (property "Value" "4,3k" (id 1) (at 99.06 106.68 90))
-    (property "Footprint" "Resistor_SMD:R_0805_2012Metric" (id 2) (at 99.06 112.268 90)
-      (effects (font (size 1.27 1.27)) hide)
-    )
+    (property "Footprint" "Resistor_SMD:R_0805_2012Metric_Pad1.20x1.40mm_HandSolder" (id 2) (at 99.06 112.268 90)
+      (effects (font (size 1.27 1.27)) hide)
+    )
